Commit message: Added lidar

File: description/robot.urdf.xacro (robot description, xacro)
@@ -3,3 +3,4 @@
     <xacro:include filename="robot_core.xacro"/>
     <xacro:include filename="gazebo_control.xacro"/>
+    <xacro:include filename="lidar.xacro"/>
 </robot>

File: description/robot_core.xacro (robot description, xacro)
@@ -12,4 +12,7 @@
     </material>
     <material name="black">
+        <color rgba="1 0 0 1"/>
+    </material>
+    <material name="red">
         <color rgba="0 0 0 1"/>
     </material>
