Commit message: Started depth camera

File: description/lidar.xacro (robot description, xacro)
@@ -1,10 +1,10 @@
 <?xml version="1.0"?>
 <robot xmlns:xacro="http://www.ros.org/wiki/xacro">
-    <joint name="lidar_joint" type="fixed">
+    <joint name="laser_joint" type="fixed">
         <parent link="chassis"/>
-        <child link="lidar_frame"/>
-        <origin xyz = "0.07 0 0.055" rpy="${pi/2} 0 ${pi/2}"/>
+        <child link="laser_frame"/>
+        <origin xyz = "0.07 0 0.055" rpy="0 0 0"/>
     </joint>
-    <link name="lidar_frame">
+    <link name="laser_frame">
         <visual>
             <geometry>
@@ -22,8 +22,9 @@
         </xacro:inertial_cylinder>
     </link>
-    <gazebo reference="lidar_frame">
-        <sensor name="lidar" type="ray">
+    <gazebo reference="laser_frame">
+        <material>Gazebo/Red</material>
+        <sensor name="laser" type="ray">
             <pose>0 0 0 0 0 0</pose>
-            <visualize>true</visualize>
+            <visualize>false</visualize>
             <update_rate>10</update_rate>
             <ray>
@@ -31,5 +32,4 @@
                     <horizontal>
                         <samples>360</samples>
-                        <resolution>1</resolution>
                         <min_angle>-3.14</min_angle>
                         <max_angle>3.14</max_angle>
@@ -39,13 +39,12 @@
                     <min>0.3</min>
                     <max>12</max>
-                    <resolution>0.01</resolution>
                 </range>
             </ray>
-            <plugin name="lidar_controller" filename="libgazebo_ros_ray_sensor.so">
+            <plugin name="laser_controller" filename="libgazebo_ros_ray_sensor.so">
                 <ros>
                     <argument>~/out:=scan</argument>
                 </ros>
-                <output_type>sensor_msgs/LidarScan</output_type>
-                <frame_name>lidar_frame</frame_name>
+                <output_type>sensor_msgs/LaserScan</output_type>
+                <frame_name>laser_frame</frame_name>
             </plugin>
         </sensor>

File: description/robot.urdf.xacro (robot description, xacro)
@@ -3,4 +3,5 @@
     <xacro:include filename="robot_core.xacro"/>
     <xacro:include filename="gazebo_control.xacro"/>
-    <xacro:include filename="lidar.xacro"/>
+    <!--<xacro:include filename="lidar.xacro"/>-->
+    <xacro:include filename="depth_camera.xacro"/>
 </robot>

Commit message: Able to map

File: description/lidar.xacro (robot description, xacro)
@@ -4,5 +4,6 @@
         <parent link="chassis"/>
         <child link="laser_frame"/>
-        <origin xyz = "0.07 0 0.055" rpy="0 0 0"/>
+        <origin xyz = "0.00 0 0.085" rpy="0 0 0"/>
+        <!-- <origin xyz = "0.00 0 0.085" rpy="0 3.14 3.14"/> -->
     </joint>
     <link name="laser_frame">
@@ -26,5 +27,5 @@
         <sensor name="laser" type="ray">
             <pose>0 0 0 0 0 0</pose>
-            <visualize>false</visualize>
+            <visualize>true</visualize>
             <update_rate>10</update_rate>
             <ray>

File: description/robot.urdf.xacro (robot description, xacro)
@@ -4,6 +4,6 @@
     <!-- <xacro:include filename="gazebo_control.xacro"/> -->
     <xacro:include filename="ros2_control.xacro"/>
-    <!-- <xacro:include filename="lidar.xacro"/> -->
+    <xacro:include filename="lidar.xacro"/>
     <!-- <xacro:include filename="camera.xacro"/> -->
-    <xacro:include filename="depth_camera.xacro"/>
+    <!-- <xacro:include filename="depth_camera.xacro"/> -->
 </robot>

File: description/robot_core.xacro (robot description, xacro)
@@ -1,7 +1,21 @@
 <?xml version="1.0"?>
-<robot xmlns:xacro="http://www.ros.org/wiki/xacro">
-    <xacro:include   filename="inertial_macros.xacro"/>
+<robot xmlns:xacro="http://www.ros.org/wiki/xacro" >
+    <xacro:include filename="inertial_macros.xacro"/>
+    <xacro:property name="chassis_length" value="0.15"/>
+    <xacro:property name="chassis_width" value="0.255"/>
+    <xacro:property name="chassis_height" value="0.06"/>
+    <xacro:property name="chassis_mass" value="1.0"/>
+    <xacro:property name="wheel_radius" value="0.075863"/>
+    <xacro:property name="wheel_thickness" value="0.015"/>
+    <xacro:property name="wheel_mass" value="0.08"/>
+    <xacro:property name="wheel_offset_x" value="0.0"/>
+    <xacro:property name="wheel_offset_y" value="0.135"/>
+    <xacro:property name="wheel_offset_z" value="0.00"/>
+    <xacro:property name="caster_wheel_radius" value="0.025"/>
+    <xacro:property name="caster_wheel_mass" value="0.01"/>
+    <xacro:property name="caster_wheel_offset_x" value="0.05"/>
+    <xacro:property name="caster_wheel_offset_z" value="${wheel_offset_z - wheel_radius + caster_wheel_radius}"/>
     <material name="white">
-        <color rgba="1 1 1 1"/>
+        <color rgba="1 1 1 1" />
     </material>
     <material name="orange">
@@ -12,8 +26,8 @@
     </material>
     <material name="black">
-        <color rgba="1 0 0 1"/>
+        <color rgba="0 0 0 1"/>
     </material>
     <material name="red">
-        <color rgba="0 0 0 1"/>
+        <color rgba="1 0 0 1"/>
     </material>
     <!-- BASE LINK -->
@@ -26,28 +40,33 @@
         <origin xyz="0 0 0" rpy="0 0 0"/>
     </joint>
+    <link name="base_footprint">
+    </link>
     <!-- CHASSIS LINK -->
     <joint name="chassis_joint" type="fixed">
         <parent link="base_link"/>
         <child link="chassis"/>
-        <origin xyz="0 0 0"/>
+        <origin xyz="${-wheel_offset_x} 0 ${-wheel_offset_z}"/>
     </joint>
     <link name="chassis">
         <visual>
+            <origin xyz="0 0 0"/>
+            <!-- <origin xyz="${chassis_length/2} 0 ${chassis_height/2}"/> -->
             <geometry>
-                <box size="0.150 0.255 .06"/>
-                <material name="white"/>
+                <box size="${chassis_length} ${chassis_width} ${chassis_height}"/>
             </geometry>
+            <material name="orange"/>
         </visual>
         <collision>
+            <origin xyz="${chassis_length/2} 0 ${chassis_height/2}"/>
             <geometry>
-                <box size="0.150 0.255 0.06"/>
+                <box size="${chassis_length} ${chassis_width} ${chassis_height}"/>
             </geometry>
         </collision>
-        <xacro:inertial_box mass="0.5" x="0.150" y="0.255" z="0.06">
-            <origin xyz="0 0 0" rpy="0 0 0"/>
+        <xacro:inertial_box mass="0.5" x="${chassis_length}" y="${chassis_width}" z="${chassis_height}">
+            <origin xyz="${chassis_length/2} 0 ${chassis_height/2}" rpy="0 0 0"/>
         </xacro:inertial_box>
     </link>
     <gazebo reference="chassis">
-        <material>Gazebo/White</material>
+        <material>Gazebo/Orange</material>
     </gazebo>
     <!-- LEFT WHEEL LINK -->
@@ -55,5 +74,5 @@
         <parent link="base_link"/>
         <child link="left_wheel"/>
-        <origin xyz="0 0.135 0" rpy="-${pi/2} 0 0"/>
+        <origin xyz="0 ${wheel_offset_y} 0" rpy="-${pi/2} 0 0" />
         <axis xyz="0 0 1"/>
     </joint>
@@ -61,5 +80,5 @@
         <visual>
             <geometry>
-                <cylinder radius="0.075375" length="0.015"/>
+                <cylinder radius="${wheel_radius}" length="${wheel_thickness}"/>
             </geometry>
             <material name="blue"/>
@@ -67,8 +86,8 @@
         <collision>
             <geometry>
-                <cylinder radius="0.075375" length="0.015"/>
+                <sphere radius="${wheel_radius}"/>
             </geometry>
         </collision>
-        <xacro:inertial_cylinder mass="0.1" length="0.015" radius="0.075375">
+        <xacro:inertial_cylinder mass="${wheel_mass}" length="${wheel_thickness}" radius="${wheel_radius}">
             <origin xyz="0 0 0" rpy="0 0 0"/>
         </xacro:inertial_cylinder>
@@ -81,5 +100,5 @@
         <parent link="base_link"/>
         <child link="right_wheel"/>
-        <origin xyz="0 -0.135 0" rpy="${pi/2} 0 0"/>
+        <origin xyz="0 ${-wheel_offset_y} 0" rpy="${pi/2} 0 0" />
         <axis xyz="0 0 -1"/>
     </joint>
@@ -87,5 +106,5 @@
         <visual>
             <geometry>
-                <cylinder radius="0.075375" length="0.015"/>
+                <cylinder radius="${wheel_radius}" length="${wheel_thickness}"/>
             </geometry>
             <material name="blue"/>
@@ -93,8 +112,8 @@
         <collision>
             <geometry>
-                <cylinder radius="0.075375" length="0.015"/>
+                <sphere radius="${wheel_radius}"/>
             </geometry>
         </collision>
-        <xacro:inertial_cylinder mass="0.1" length="0.015" radius="0.075375">
+        <xacro:inertial_cylinder mass="${wheel_mass}" length="${wheel_thickness}" radius="${wheel_radius}">
             <origin xyz="0 0 0" rpy="0 0 0"/>
         </xacro:inertial_cylinder>
@@ -103,54 +122,55 @@
         <material>Gazebo/Blue</material>
     </gazebo>
-    <!-- CASTER WHEELS -->
-    <joint name="caster_wheel_front_joint" type="fixed">
+    <!-- CASTER WHEEL LINK -->
+    <joint name="caster_wheel_joint" type="fixed">
         <parent link="chassis"/>
-        <child link="caster_wheel_front"/>
-        <origin xyz="0.05 0 -0.05"/>
+        <child link="caster_wheel"/>
+        <origin xyz="${caster_wheel_offset_x} 0 ${caster_wheel_offset_z}"/>
     </joint>
-    <link name="caster_wheel_front">
+    <link name="caster_wheel">
         <visual>
             <geometry>
-                <sphere radius="0.025"/>
+                <sphere radius="${caster_wheel_radius}"/>
             </geometry>
-            <material name="black"/>
+            <material name="white"/>
         </visual>
         <collision>
             <geometry>
-                <sphere radius="0.025"/>
+                <sphere radius="${caster_wheel_radius}"/>
             </geometry>
         </collision>
-        <xacro:inertial_sphere mass="0.1" radius="0.025">
+        <xacro:inertial_sphere mass="${caster_wheel_mass}" radius="${caster_wheel_radius}">
             <origin xyz="0 0 0" rpy="0 0 0"/>
         </xacro:inertial_sphere>
     </link>
-    <gazebo reference="caster_wheel_front">
-        <material>Gazebo/Black</material>
+    <gazebo reference="caster_wheel">
+        <material>Gazebo/White</material>
         <mu1 value="0.001"/>
         <mu2 value="0.001"/>
     </gazebo>
-    <joint name="caster_wheel_back_joint" type="fixed">
+    <!-- CASTER WHEEL LINK -->
+    <joint name="caster_wheel_joint_2" type="fixed">
         <parent link="chassis"/>
-        <child link="caster_wheel_back"/>
-        <origin xyz="-0.05 0 -0.05"/>
+        <child link="caster_wheel_2"/>
+        <origin xyz="${-caster_wheel_offset_x} 0 ${caster_wheel_offset_z}"/>
     </joint>
-    <link name="caster_wheel_back">
+    <link name="caster_wheel_2">
         <visual>
             <geometry>
-                <sphere radius="0.025"/>
+                <sphere radius="${caster_wheel_radius}"/>
             </geometry>
-            <material name="black"/>
+            <material name="white"/>
         </visual>
         <collision>
             <geometry>
-                <sphere radius="0.025"/>
+                <sphere radius="${caster_wheel_radius}"/>
             </geometry>
         </collision>
-        <xacro:inertial_sphere mass="0.1" radius="0.025">
+        <xacro:inertial_sphere mass="${caster_wheel_mass}" radius="${caster_wheel_radius}">
             <origin xyz="0 0 0" rpy="0 0 0"/>
         </xacro:inertial_sphere>
     </link>
-    <gazebo reference="caster_wheel_back">
-        <material>Gazebo/Black</material>
+    <gazebo reference="caster_wheel_2">
+        <material>Gazebo/White</material>
         <mu1 value="0.001"/>
         <mu2 value="0.001"/>

File: description/ros2_control.xacro (robot description, xacro)
@@ -8,20 +8,20 @@
         </hardware>
         <joint name="left_wheel_joint">
-        <command_interface name="velocity"/>
-        <state_interface name="position"/>
-        <param name="address">128</param>
-        <!--motor types must be one of M1 or M2-->
-        <param name="motor_type">M1</param>
-        <!-- Number of encoder ticks per wheel rotation -->
-        <param name="qppr">386</param>
+            <command_interface name="velocity"/>
+            <state_interface name="position"/>
+            <param name="address">128</param>
+            <!--motor types must be one of M1 or M2-->
+            <param name="motor_type">M1</param>
+            <!-- Number of encoder ticks per wheel rotation -->
+            <param name="qppr">400</param>
         </joint>
         <joint name="right_wheel_joint">
-        <command_interface name="velocity"/>
-        <state_interface name="position"/>
-        <param name="address">128</param>
-        <!--motor types must be one of M1 or M2-->
-        <param name="motor_type">M2</param>
-        <!-- Number of encoder ticks per wheel rotation -->
-        <param name="qppr">386</param>
+            <command_interface name="velocity"/>
+            <state_interface name="position"/>
+            <param name="address">128</param>
+            <!--motor types must be one of M1 or M2-->
+            <param name="motor_type">M2</param>
+            <!-- Number of encoder ticks per wheel rotation -->
+            <param name="qppr">400</param>
         </joint>
     </ros2_control>

Commit message: New body design

File: description/lidar.xacro (robot description, xacro)
@@ -4,5 +4,5 @@
         <parent link="chassis"/>
         <child link="laser_frame"/>
-        <origin xyz = "0.00 0 0.085" rpy="0 0 0"/>
+        <origin xyz = "0.00 0 0.054" rpy="0 0 0"/>
         <!-- <origin xyz = "0.00 0 0.085" rpy="0 3.14 3.14"/> -->
     </joint>
@@ -10,5 +10,5 @@
         <visual>
             <geometry>
-                <cylinder radius="0.0305" length="0.026"/>
+                <cylinder radius="0.035" length="0.024"/>
             </geometry>
             <material name="red"/>
@@ -16,8 +16,8 @@
         <collision>
             <geometry>
-                <cylinder radius="0.0305" length="0.026"/>
+                <cylinder radius="0.035" length="0.024"/>
             </geometry>
         </collision>
-        <xacro:inertial_cylinder mass="0.1" length="0.026" radius="0.0305">
+        <xacro:inertial_cylinder mass="0.1" length="0.024" radius="0.035">
             <origin xyz="0 0 0" rpy="0 0 0"/>
         </xacro:inertial_cylinder>
@@ -52,2 +52,26 @@
     </gazebo>
 </robot>
+<!-- <?xml version="1.0"?>
+<robot xmlns:xacro="http://www.ros.org/wiki/xacro">
+    <joint name="laser_joint" type="fixed">
+        <parent link="chassis"/>
+        <child link="laser_frame"/>
+        <origin xyz = "0.00 0 0.115" rpy="0 0 0"/>
+    </joint>
+    <link name="laser_frame">
+        <visual>
+            <geometry>
+                <cylinder radius="0.0225" length="0.0225"/>
+            </geometry>
+            <material name="red"/>
+        </visual>
+        <collision>
+            <geometry>
+                <cylinder radius="0.0225" length="0.0225"/>
+            </geometry>
+        </collision>
+        <xacro:inertial_cylinder mass="0.1" length="0.0225" radius="0.0225">
+            <origin xyz="0 0 0" rpy="0 0 0"/>
+        </xacro:inertial_cylinder>
+    </link>
+</robot> -->

File: description/robot_core.xacro (robot description, xacro)
@@ -2,17 +2,16 @@
 <robot xmlns:xacro="http://www.ros.org/wiki/xacro" >
     <xacro:include filename="inertial_macros.xacro"/>
-    <xacro:property name="chassis_length" value="0.15"/>
-    <xacro:property name="chassis_width" value="0.255"/>
-    <xacro:property name="chassis_height" value="0.06"/>
+    <xacro:property name="chassis_radius" value="0.17"/>
+    <xacro:property name="chassis_height" value="0.08535"/>
     <xacro:property name="chassis_mass" value="1.0"/>
-    <xacro:property name="wheel_radius" value="0.075863"/>
+    <xacro:property name="wheel_radius" value="0.0415"/>
     <xacro:property name="wheel_thickness" value="0.015"/>
     <xacro:property name="wheel_mass" value="0.08"/>
     <xacro:property name="wheel_offset_x" value="0.0"/>
-    <xacro:property name="wheel_offset_y" value="0.135"/>
-    <xacro:property name="wheel_offset_z" value="0.00"/>
-    <xacro:property name="caster_wheel_radius" value="0.025"/>
+    <xacro:property name="wheel_offset_y" value="0.14265"/>
+    <xacro:property name="wheel_offset_z" value="-0.01"/>
+    <xacro:property name="caster_wheel_radius" value="0.00925"/>
     <xacro:property name="caster_wheel_mass" value="0.01"/>
-    <xacro:property name="caster_wheel_offset_x" value="0.05"/>
+    <xacro:property name="caster_wheel_offset_x" value="0.139"/>
     <xacro:property name="caster_wheel_offset_z" value="${wheel_offset_z - wheel_radius + caster_wheel_radius}"/>
     <material name="white">
@@ -51,19 +50,19 @@
         <visual>
             <origin xyz="0 0 0"/>
-            <!-- <origin xyz="${chassis_length/2} 0 ${chassis_height/2}"/> -->
+            <!-- <origin xyz="${chassis_radius} 0 ${chassis_height/2}"/> -->
             <geometry>
-                <box size="${chassis_length} ${chassis_width} ${chassis_height}"/>
+                <cylinder radius="${chassis_radius}" length="${chassis_height}"/>
             </geometry>
             <material name="orange"/>
         </visual>
         <collision>
-            <origin xyz="${chassis_length/2} 0 ${chassis_height/2}"/>
+            <origin xyz="${chassis_radius} 0 ${chassis_height/2}"/>
             <geometry>
-                <box size="${chassis_length} ${chassis_width} ${chassis_height}"/>
+                <cylinder radius="${chassis_radius}" length="${chassis_height}"/>
             </geometry>
         </collision>
-        <xacro:inertial_box mass="0.5" x="${chassis_length}" y="${chassis_width}" z="${chassis_height}">
-            <origin xyz="${chassis_length/2} 0 ${chassis_height/2}" rpy="0 0 0"/>
-        </xacro:inertial_box>
+        <xacro:inertial_cylinder mass="0.5" length="${chassis_height}" radius="${chassis_radius}">
+            <origin xyz="${chassis_radius} 0 ${chassis_height/2}" rpy="0 0 0"/>
+        </xacro:inertial_cylinder>
     </link>
     <gazebo reference="chassis">
